File: Ampli_Audio.kicad_sch (KiCad schematic)
At the start: 51 parts, among them J2 Conn_01x02, J3 Conn_01x03, Q1 2N2907, Q10 TIP32, Q11 BD138, Q12 TIP31, Q13 2N2222, Q2 2N2907, Q3 2N2907, Q4 2N2222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

Commit message: Placement composants sur PCB
Parts:
- C1: footprint CmpAmpliAudioTR:CP_Radial_D12.5mm_P5.00mm -> CmpAmpliAudioTR:CP_Radial_D8.0mm_P5.00mm
- C3: footprint CmpAmpliAudioTR:C_Rect_L7.2mm_W3.5mm_P5.00mm_FKS2_FKP2_MKS2_MKP2 -> CmpAmpliAudioTR:CP_Radial_D8.0mm_P5.00mm
- C4, C6: footprint (none) -> CmpAmpliAudioTR:CP_Radial_D8.0mm_P5.00mm
- C8: footprint CmpAmpliAudioTR:C_Rect_L7.2mm_W3.5mm_P5.00mm_FKS2_FKP2_MKS2_MKP2 -> CmpAmpliAudioTR:CP_Radial_D12.5mm_P5.00mm
- Dz1: footprint (none) -> CmpAmpliAudioTR:D_DO-35_SOD27_P10.16mm_Horizontal
- RV1: footprint CmpAmpliAudioTR:Heatsink_Fischer_SK104-STC-STIC_35x13mm_2xDrill2.5mm -> CmpAmpliAudioTR:Potentiometer_Bourns_3296W_Vertical
- U1: footprint CmpAmpliAudioTR:Potentiometer_Bourns_3296W_Vertical -> CmpAmpliAudioTR:Relais_112LMH2
Changed lines of the file:
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@@
       (effects (font (size 1.27 1.27)) (justify left))
     )
-    (property "Footprint" "" (id 2) (at 55.5752 179.07 0)
+    (property "Footprint" "CmpAmpliAudioTR:CP_Radial_D8.0mm_P5.00mm" (id 2) (at 55.5752 179.07 0)
       (effects (font (size 1.27 1.27)) hide)
     )
@@
       (effects (font (size 1.27 1.27)) (justify left))
     )
-    (property "Footprint" "" (id 2) (at 63.5 34.29 0)
+    (property "Footprint" "CmpAmpliAudioTR:D_DO-35_SOD27_P10.16mm_Horizontal" (id 2) (at 63.5 34.29 0)
       (effects (font (size 1.27 1.27)) hide)
     )
@@
       (effects (font (size 1.27 1.27)) (justify right))
     )
-    (property "Footprint" "CmpAmpliAudioTR:Heatsink_Fischer_SK104-STC-STIC_35x13mm_2xDrill2.5mm" (id 2) (at 118.11 72.39 0)
+    (property "Footprint" "CmpAmpliAudioTR:Potentiometer_Bourns_3296W_Vertical" (id 2) (at 118.11 72.39 0)
       (effects (font (size 1.27 1.27)) hide)
     )
@@
       (effects (font (size 1.27 1.27)) (justify left))
     )
-    (property "Footprint" "CmpAmpliAudioTR:C_Rect_L7.2mm_W3.5mm_P5.00mm_FKS2_FKP2_MKS2_MKP2" (id 2) (at 194.0052 52.07 0)
+    (property "Footprint" "CmpAmpliAudioTR:CP_Radial_D12.5mm_P5.00mm" (id 2) (at 194.0052 52.07 0)
       (effects (font (size 1.27 1.27)) hide)
     )
@@
       (effects (font (size 1.27 1.27)) (justify left))
     )
-    (property "Footprint" "CmpAmpliAudioTR:C_Rect_L7.2mm_W3.5mm_P5.00mm_FKS2_FKP2_MKS2_MKP2" (id 2) (at 247.3452 130.81 0)
+    (property "Footprint" "CmpAmpliAudioTR:CP_Radial_D8.0mm_P5.00mm" (id 2) (at 247.3452 130.81 0)
       (effects (font (size 1.27 1.27)) hide)
     )
@@
       (effects (font (size 1.27 1.27)) (justify left))
     )
-    (property "Footprint" "" (id 2) (at 55.5752 161.29 0)
+    (property "Footprint" "CmpAmpliAudioTR:CP_Radial_D8.0mm_P5.00mm" (id 2) (at 55.5752 161.29 0)
       (effects (font (size 1.27 1.27)) hide)
     )
@@
     (property "Reference" "U1" (id 0) (at 233.68 74.93 90))
     (property "Value" "Relay_1CT" (id 1) (at 233.68 77.47 90))
-    (property "Footprint" "CmpAmpliAudioTR:Potentiometer_Bourns_3296W_Vertical" (id 2) (at 233.68 87.63 0)
+    (property "Footprint" "CmpAmpliAudioTR:Relais_112LMH2" (id 2) (at 233.68 87.63 0)
       (effects (font (size 1.27 1.27)) hide)
     )
@@
     (property "Reference" "C1" (id 0) (at 45.72 93.98 90))
     (property "Value" "47u" (id 1) (at 45.72 101.6 90))
-    (property "Footprint" "CmpAmpliAudioTR:CP_Radial_D12.5mm_P5.00mm" (id 2) (at 41.91 98.7552 0)
+    (property "Footprint" "CmpAmpliAudioTR:CP_Radial_D8.0mm_P5.00mm" (id 2) (at 41.91 98.7552 0)
       (effects (font (size 1.27 1.27)) hide)
     )
@@
     )
     (path "/b752bda3-13c7-4a57-9e66-fac5ed0b3f84"
-      (reference "C1") (unit 1) (value "47u") (footprint "CmpAmpliAudioTR:CP_Radial_D12.5mm_P5.00mm")
+      (reference "C1") (unit 1) (value "47u") (footprint "CmpAmpliAudioTR:CP_Radial_D8.0mm_P5.00mm")
     )
     (path "/8138a812-ad1f-4669-b46d-d687671a4278"
@@
     )
     (path "/7e366d80-6712-40b4-ad25-6f0ee9e94346"
-      (reference "C3") (unit 1) (value "100u") (footprint "CmpAmpliAudioTR:C_Rect_L7.2mm_W3.5mm_P5.00mm_FKS2_FKP2_MKS2_MKP2")
+      (reference "C3") (unit 1) (value "100u") (footprint "CmpAmpliAudioTR:CP_Radial_D8.0mm_P5.00mm")
     )
     (path "/881151d5-15ed-4355-a69f-6abefa3c2028"
-      (reference "C4") (unit 1) (value "10u") (footprint "")
+      (reference "C4") (unit 1) (value "10u") (footprint "CmpAmpliAudioTR:CP_Radial_D8.0mm_P5.00mm")
     )
     (path "/1409a2a3-4f15-4c7d-a042-5fc36dcf732d"
@@
     )
     (path "/3bfcbcca-b58d-4929-876d-00863865e078"
-      (reference "C6") (unit 1) (value "10u") (footprint "")
+      (reference "C6") (unit 1) (value "10u") (footprint "CmpAmpliAudioTR:CP_Radial_D8.0mm_P5.00mm")
     )
     (path "/8e1309e7-40cd-4875-a50b-909fb696e690"
@@
     )
     (path "/69d3cba1-3708-4aa2-817b-6cc6464f3ce1"
-      (reference "C8") (unit 1) (value "470u") (footprint "CmpAmpliAudioTR:C_Rect_L7.2mm_W3.5mm_P5.00mm_FKS2_FKP2_MKS2_MKP2")
+      (reference "C8") (unit 1) (value "470u") (footprint "CmpAmpliAudioTR:CP_Radial_D12.5mm_P5.00mm")
     )
     (path "/d97b9dbf-88ee-465c-9f97-babb7d5604e4"
@@
     )
     (path "/422938f0-c42f-4637-ad9a-bedde43edf63"
-      (reference "Dz1") (unit 1) (value "BZX55C5V1") (footprint "")
+      (reference "Dz1") (unit 1) (value "BZX55C5V1") (footprint "CmpAmpliAudioTR:D_DO-35_SOD27_P10.16mm_Horizontal")
     )
     (path "/9111d637-58c6-40e6-ad60-d176ee7daaa6"
@@
     )
     (path "/5ec1e6f2-cb34-40f1-ad7b-98189ce7c827"
-      (reference "RV1") (unit 1) (value "R_POT") (footprint "CmpAmpliAudioTR:Heatsink_Fischer_SK104-STC-STIC_35x13mm_2xDrill2.5mm")
+      (reference "RV1") (unit 1) (value "R_POT") (footprint "CmpAmpliAudioTR:Potentiometer_Bourns_3296W_Vertical")
     )
     (path "/b5f72fc0-39c7-41aa-a3d9-34ddb2e446be"
@@
     )
     (path "/a8523b99-522b-44c7-a5af-9ab9ecc4c598"
-      (reference "U1") (unit 1) (value "Relay_1CT") (footprint "CmpAmpliAudioTR:Potentiometer_Bourns_3296W_Vertical")
+      (reference "U1") (unit 1) (value "Relay_1CT") (footprint "CmpAmpliAudioTR:Relais_112LMH2")
     )
     (path "/1e17fc22-e279-4742-81e3-1993a926b45c"

Commit message: Correction & Routage
Connections:
- net +12V: now also Q10.3 (E); no longer Q10.2 (C)
- net GND: now also J2.1 (Pin_1); no longer J2.2 (Pin_2)
- net at Q9.1 (E), R11.1: now also Q10.2 (C); no longer Q10.3 (E)
- net at U1.c2: now also J2.2 (Pin_2); no longer J2.1 (Pin_1)
Changed lines of the file:
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@@
     (pin "1")
   )
-  (symbol (lib_id "Device:Q_PNP_BCE") (at 163.83 48.26 0) (unit 1)
+  (symbol (lib_id "Device:Q_PNP_BCE") (at 163.83 48.26 0) (mirror x) (unit 1)
     (in_bom yes) (on_board yes)
-    (property "Reference" "Q10" (id 0) (at 160.02 40.64 0)
+    (property "Reference" "Q10" (id 0) (at 158.75 44.45 0)
       (effects (font (size 1.27 1.27)) (justify left))
     )
-    (property "Value" "TIP32" (id 1) (at 160.02 43.18 0)
+    (property "Value" "TIP32" (id 1) (at 158.75 41.91 0)
       (effects (font (size 1.27 1.27)) (justify left))
     )
-    (property "Footprint" "CmpAmpliAudioTR:TO-220-3_Vertical" (id 2) (at 168.91 45.72 0)
+    (property "Footprint" "CmpAmpliAudioTR:TO-220-3_Vertical" (id 2) (at 168.91 50.8 0)
       (effects (font (size 1.27 1.27)) hide)
     )
@@
     (pin "3")
   )
-  (symbol (lib_id "Connector_Generic:Conn_01x02") (at 261.62 82.55 0) (unit 1)
+  (symbol (lib_id "Connector_Generic:Conn_01x02") (at 261.62 85.09 0) (mirror x) (unit 1)
     (in_bom yes) (on_board yes) (fields_autoplaced)
-    (property "Reference" "J2" (id 0) (at 264.16 82.5499 0)
-      (effects (font (size 1.27 1.27)) (justify left))
-    )
-    (property "Value" "Conn_01x02" (id 1) (at 264.16 85.0899 0)
-      (effects (font (size 1.27 1.27)) (justify left))
-    )
-    (property "Footprint" "CmpAmpliAudioTR:PhoenixContact_MSTBVA_2,5_2-G-5,08_1x02_P5.08mm_Vertical" (id 2) (at 261.62 82.55 0)
+    (property "Reference" "J2" (id 0) (at 261.62 76.2 0))
+    (property "Value" "Conn_01x02" (id 1) (at 261.62 78.74 0))
+    (property "Footprint" "CmpAmpliAudioTR:PhoenixContact_MSTBVA_2,5_2-G-5,08_1x02_P5.08mm_Vertical" (id 2) (at 261.62 85.09 0)
       (effects (font (size 1.27 1.27)) hide)
     )
-    (property "Datasheet" "~" (id 3) (at 261.62 82.55 0)
+    (property "Datasheet" "~" (id 3) (at 261.62 85.09 0)
       (effects (font (size 1.27 1.27)) hide)
     )
