File: Ampli_Audio.kicad_pcb (KiCad board)
At the start: 2 copper layers, 110 x 100 mm, 51 parts, among them J2 Conn_01x02, J3 Conn_01x03, Q1 2N2907, Q10 TIP32, Q11 BD138, Q12 TIP31, Q13 2N2222, Q2 2N2907, Q3 2N2907, Q4 2N2222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

Commit message: Correction & Routage
Parts:
- moved C5 52.9 mm to (73.7, 34.9)
- moved C7 51.8 mm to (125.7, 41.2)
- moved C4 34.0 mm to (83.2, 34.8)
- moved C6 33.0 mm to (116.2, 41.1)
- moved R7 10.2 mm to (31.8, 72.4), turned to -90 degrees
- moved C3 1.27 mm to (124.6, 51.4)
Connections:
- J2 pad 1: Net-(J2-Pad1) -> GND
- J2 pad 2: GND -> Net-(J2-Pad2)
- Q10 pad 2: +12V -> Net-(Q10-Pad2)
- Q10 pad 3: Net-(Q10-Pad3) -> +12V
- Q9 pad 1: Net-(Q10-Pad3) -> Net-(Q10-Pad2)
- R11 pad 1: Net-(Q10-Pad3) -> Net-(Q10-Pad2)
- U1 pad c2: Net-(J2-Pad1) -> Net-(J2-Pad2)
Routing:
- net GND: track 0.00 -> 350.0 mm
- net +12V: track 0.00 -> 244.1 mm
- net -12V: track 0.00 -> 142.2 mm
- net Net-(Q1-Pad1): track 0.00 -> 106.8 mm
- net Net-(R11-Pad2): track 0.00 -> 86.2 mm, vias 0 -> 2
- net Net-(C2-Pad2): track 0.00 -> 84.0 mm
- net Net-(R10-Pad2): track 0.00 -> 79.5 mm
- net Net-(C2-Pad1): track 0.00 -> 48.1 mm
- net Net-(Q2-Pad2): track 0.00 -> 47.0 mm
- net Net-(Q11-Pad1): track 0.00 -> 45.1 mm
- net Net-(Q6-Pad3): track 0.00 -> 39.0 mm
- net Net-(Q10-Pad2): track 0.00 -> 32.7 mm
- net Net-(Q6-Pad2): track 0.00 -> 29.1 mm
- net Net-(C1-Pad1): track 0.00 -> 28.1 mm
- net Net-(J2-Pad2): track 0.00 -> 24.8 mm
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- added copper zone on B.Cu, net GND

Commit message: Révisions PCB
Parts:
- added REF**: INSA_Toulouse, CmpAmpliAudioTR:INSA_Toulouse, B.Cu at (124.5, 99.7)
- moved U2 0.20 mm to (55.9, 125.5)
Routing:
- net GND: track 350.0 -> 0.00 mm
- net +12V: track 244.1 -> 239.5 mm
- net Net-(Q2-Pad2): track 47.0 -> 42.9 mm
- net Net-(Q11-Pad1): track 45.1 -> 47.9 mm
- net Net-(R11-Pad2): track 86.2 -> 87.8 mm
- net -12V: track 142.2 -> 143.5 mm
- net Net-(C3-Pad1): track 12.0 -> 12.8 mm
- net Net-(Q10-Pad2): track 32.7 -> 31.9 mm
Other:
- board text added: "Ampli Audio"
- board text added: "Cyprien Heusse S2 2022"
